File: Hardware/Schematic.sch (EAGLE design)
At the start: 105 parts, among them IC1 BQ25180YBGR, IC2 DRV2605YZFR, IC3 BMA421, IC9 RT6160AWSC, J2 TC2030-IDC, J3 503480-2400, J4 KH-TYPE-C-16P, Q1 20V/4.2A/52mΩ/1.4W, Q3 SI1308EDL-T1-GE3, U1 NRF52840_QF, U3 MAX17048G+T10, X1 32MHz, X2 32.768kHz

Commit message: Add files via upload
Parts:
- C39: device InkTime_v5:NORDIC_NRF_3_CAPACITOR_0201_L -> InkTime_v5:NORDIC_NRF_3_CAPACITOR_0402_N
Connections:
- net N$13 renamed P0.00/XL1
- net N$14 renamed P0.01/XL2
