File: Hardware/PCB.brd (EAGLE design)
At the start: 46 x 35 mm, 105 parts, among them IC1 BQ25180YBGR, IC2 DRV2605YZFR, IC3 BMA421, IC9 RT6160AWSC, J2 TC2030-IDC, J3 503480-2400, J4 KH-TYPE-C-16P, Q1 20V/4.2A/52mΩ/1.4W, Q3 SI1308EDL-T1-GE3, U1 NRF52840_QF, U3 MAX17048G+T10, X1 32MHz, X2 32.768kHz

Commit message: Add files via upload
Parts:
- C39: device InkTime_v5:NORDIC_NRF_3_RESC0201_L -> InkTime_v5:NORDIC_NRF_3_RESC0402_N
- moved ANT1 13.7 mm to (16.3, 12.9), turned to 180 degrees
- moved TP_SWDCLK 8.65 mm to (21.0, 4.92)
Connections:
- net N$13 renamed P0.00/XL1
- net N$14 renamed P0.01/XL2
Routing:
- net RF: track 5.79 -> 19.1 mm
- net SWDCLK: track 32.6 -> 24.7 mm
Other:
- outline, holes or cut-outs redrawn
